File: SW-SMART-SIX-HIGH.kicad_pcb (KiCad board)
At the start: 2 copper layers, 72 x 69 mm, 53 parts, among them J1 SWLINK, J2 USART1, J3 POWER OUT, J4 POWER IN, SW0 BTS7002-1EPP, SW1 BTS7002-1EPP, SW2 BTS7002-1EPP, U1 STM32G0B1KBTx, U4 MCP2562-E-SN

Commit message: lots of work to do!
Parts:
- removed CVIN1: 10u, Capacitor_SMD:C_1206_3216Metric_Pad1.33x1.80mm_HandSolder
- removed VR5V0: NCV1117ST50, PCM_SparkFun-Semiconductor-Standard:SOT-223-3_TabPin2
- added C15: 100n, Capacitor_SMD:C_0603_1608Metric_Pad1.08x0.95mm_HandSolder, F.Cu at (61.2, 110.6)
- added CIN1: 10u, Capacitor_SMD:C_1210_3225Metric_Pad1.33x2.70mm_HandSolder, F.Cu at (66.4, 121.1)
- added CIN2: 100n, Capacitor_SMD:C_0603_1608Metric_Pad1.08x0.95mm_HandSolder, F.Cu at (61.2, 113.1)
- added COUT3: 10u, Capacitor_SMD:C_0805_2012Metric_Pad1.18x1.45mm_HandSolder, F.Cu at (74.1, 110.9)
- added COUT4: 10u, Capacitor_SMD:C_0805_2012Metric_Pad1.18x1.45mm_HandSolder, F.Cu at (74.1, 113.9)
- added COUT5: 10n, Capacitor_SMD:C_0603_1608Metric_Pad1.08x0.95mm_HandSolder, F.Cu at (116.3, 106.3)
- added COUT6: 10n, Capacitor_SMD:C_0603_1608Metric_Pad1.08x0.95mm_HandSolder, F.Cu at (116.3, 108.8)
- added COUT7: 10n, Capacitor_SMD:C_0603_1608Metric_Pad1.08x0.95mm_HandSolder, F.Cu at (116.3, 111.3)
- added J5: POWER OUT, TerminalBlock_Phoenix:TerminalBlock_Phoenix_MKDS-3-5-5.08_1x05_P5.08mm_Horizontal, F.Cu at (180.2, 87.1)
- added L1: 8.2 uH 55.2 mOhm, SamacSys_Parts:SRP5030HMT2R2M, F.Cu at (67.5, 114.2)
- added R13: 4K7, Resistor_SMD:R_0603_1608Metric_Pad0.98x0.95mm_HandSolder, F.Cu at (116.3, 113.9)
- added R14: 4K7, Resistor_SMD:R_0603_1608Metric_Pad0.98x0.95mm_HandSolder, F.Cu at (116.3, 116.4)
- added R15: 10K, Resistor_SMD:R_0603_1608Metric_Pad0.98x0.95mm_HandSolder, F.Cu at (116.3, 118.9)
- added R16: 4K7, Resistor_SMD:R_0603_1608Metric_Pad0.98x0.95mm_HandSolder, F.Cu at (116.3, 121.4)
- added R17: 4K7, Resistor_SMD:R_0603_1608Metric_Pad0.98x0.95mm_HandSolder, F.Cu at (116.3, 123.9)
- added R18: 10K, Resistor_SMD:R_0603_1608Metric_Pad0.98x0.95mm_HandSolder, F.Cu at (120.7, 106.3)
- added R19: 4K7, Resistor_SMD:R_0603_1608Metric_Pad0.98x0.95mm_HandSolder, F.Cu at (120.7, 108.8)
- added R20: 4K7, Resistor_SMD:R_0603_1608Metric_Pad0.98x0.95mm_HandSolder, F.Cu at (120.7, 111.3)
- added R21: 10K, Resistor_SMD:R_0603_1608Metric_Pad0.98x0.95mm_HandSolder, F.Cu at (120.7, 113.9)
- added R22: 1K0, Resistor_SMD:R_0603_1608Metric_Pad0.98x0.95mm_HandSolder, F.Cu at (120.7, 116.4)
- added R23: 1K0, Resistor_SMD:R_0603_1608Metric_Pad0.98x0.95mm_HandSolder, F.Cu at (120.7, 118.9)
- added R24: 1K0, Resistor_SMD:R_0603_1608Metric_Pad0.98x0.95mm_HandSolder, F.Cu at (120.7, 121.4)
- added RFBT1: 115K, Resistor_SMD:R_0603_1608Metric_Pad0.98x0.95mm_HandSolder, F.Cu at (61.2, 115.6)
- added RGND3: 47R, Resistor_SMD:R_0603_1608Metric_Pad0.98x0.95mm_HandSolder, F.Cu at (120.7, 123.9)
- added RGND4: 47R, Resistor_SMD:R_0603_1608Metric_Pad0.98x0.95mm_HandSolder, F.Cu at (125.0, 106.3)
- added RGND5: 47R, Resistor_SMD:R_0603_1608Metric_Pad0.98x0.95mm_HandSolder, F.Cu at (125.0, 108.8)
- added RPD3: 47K, Resistor_SMD:R_0603_1608Metric_Pad0.98x0.95mm_HandSolder, F.Cu at (125.0, 111.3)
- added RPD4: 47K, Resistor_SMD:R_0603_1608Metric_Pad0.98x0.95mm_HandSolder, F.Cu at (125.0, 113.9)
- added RPD5: 47K, Resistor_SMD:R_0603_1608Metric_Pad0.98x0.95mm_HandSolder, F.Cu at (125.0, 116.4)
- added RRFBB1: 22K1, Resistor_SMD:R_0603_1608Metric_Pad0.98x0.95mm_HandSolder, F.Cu at (61.2, 118.1)
- added SW3: BTS7002-1EPP, SamacSys_Parts:SOP65P600X115-15N, F.Cu at (180.6, 106.5)
- added SW4: BTS7002-1EPP, SamacSys_Parts:SOP65P600X115-15N, F.Cu at (170.1, 106.5)
- added SW5: BTS7002-1EPP, SamacSys_Parts:SOP65P600X115-15N, F.Cu at (159.8, 106.5)
- added U3: LMR54410, Package_TO_SOT_SMD:SOT-23-6, F.Cu at (72.0, 121.3)
- moved H1 159.0 mm to (245.0, 74.8), turned to -90 degrees
- moved J3 134.4 mm to (233.2, 87.5), turned to 180 degrees
- moved COUT2 125.7 mm to (238.0, 103.6), turned to -90 degrees
- moved CVS2 120.5 mm to (237.8, 110.1), turned to -90 degrees
- moved SW2 119.0 mm to (234.2, 106.5), turned to 90 degrees
- moved R7 117.2 mm to (236.2, 112.2), turned to 90 degrees
- moved RPD2 117.0 mm to (230.5, 103.6), turned to 90 degrees
- moved H3 116.9 mm to (245.0, 135.8), turned to -90 degrees
- moved H2 115.5 mm to (188.0, 74.8), turned to -90 degrees
- moved R6 115.4 mm to (234.8, 112.2), turned to 90 degrees
- moved R2 113.5 mm to (233.2, 112.2), turned to 90 degrees
- moved COUT1 112.8 mm to (226.8, 103.6), turned to -90 degrees
- moved R1 111.7 mm to (231.8, 112.2), turned to 90 degrees
- moved RGND2 109.9 mm to (230.2, 112.2), turned to -90 degrees
- moved CVS1 107.3 mm to (226.8, 110.1), turned to -90 degrees
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Connections:
- net /SW0DEN renamed /SWDEN0
- net /SW0IN renamed /SWIN0
- net /SW0IS renamed /SWIS0
- net /SW0IS_PD renamed /SWIS_PD0
- net /SW1DEN renamed /SWDEN1
- net /SW1IN renamed /SWIN1
- net /SW1IS renamed /SWIS1
- net /SW1IS_PD renamed /SWIS_PD1
- net /SW2DEN renamed /SWDEN2
- net /SW2IN renamed /SWIN2
- net /SW2IS renamed /SWIS2
- net /SW2IS_PD renamed /SWIS_PD2
- COUT0 pad 1: /SW0OUT -> /SWOUT0
- COUT1 pad 1: /SW1OUT -> /SWOUT1
- COUT2 pad 1: /SW2OUT -> /SWOUT2
- J3 pad 1: /SW2OUT -> unconnected-(J3-Pin_1-Pad1)
- J3 pad 3: /SW1OUT -> unconnected-(J3-Pin_3-Pad3)
- J3 pad 5: /SW0OUT -> unconnected-(J3-Pin_5-Pad5)
- RPD0 pad 2: /SW0OUT -> /SWOUT0
- RPD1 pad 2: /SW1OUT -> /SWOUT1
- RPD2 pad 2: /SW2OUT -> /SWOUT2
- SW0 pad 10: /SW0OUT -> /SWOUT0
- SW0 pad 12: /SW0OUT -> /SWOUT0
- SW0 pad 13: /SW0OUT -> /SWOUT0
- SW0 pad 14: /SW0OUT -> /SWOUT0
- SW0 pad 8: /SW0OUT -> /SWOUT0
- SW0 pad 9: /SW0OUT -> /SWOUT0
- SW1 pad 10: /SW1OUT -> /SWOUT1
- SW1 pad 12: /SW1OUT -> /SWOUT1
- SW1 pad 13: /SW1OUT -> /SWOUT1
- SW1 pad 14: /SW1OUT -> /SWOUT1
- SW1 pad 8: /SW1OUT -> /SWOUT1
- SW1 pad 9: /SW1OUT -> /SWOUT1
- SW2 pad 10: /SW2OUT -> /SWOUT2
- SW2 pad 12: /SW2OUT -> /SWOUT2
- SW2 pad 13: /SW2OUT -> /SWOUT2
- SW2 pad 14: /SW2OUT -> /SWOUT2
- SW2 pad 8: /SW2OUT -> /SWOUT2
- SW2 pad 9: /SW2OUT -> /SWOUT2
Routing:
- net +5V: track 62.3 -> 47.7 mm
- net GND: track 99.5 -> 90.3 mm, vias 24 -> 23
- net +12V: track 3.03 -> 0.00 mm
- net /SWIS0: track 24.6 -> 23.9 mm
- net /CAN_L: track 18.5 -> 18.0 mm
- net /SWOUT2: vias 0 -> 20
- net /SWOUT1: vias 0 -> 20
- net /SWOUT0: vias 0 -> 21
- net /SW2OUT: vias 20 -> 0
- net /SW1OUT: vias 20 -> 0
- net /SW0OUT: vias 21 -> 0
- added copper zone on B.Cu, net /SWOUT0
- added copper zone on F.Cu, net /SWOUT0
- added copper zone on B.Cu, net /SWOUT1
- added copper zone on F.Cu, net /SWOUT1
- added copper zone on B.Cu, net /SWOUT2
- added copper zone on F.Cu, net /SWOUT2
- removed copper zone on B.Cu, net /SW0OUT
- removed copper zone on F.Cu, net /SW0OUT
- removed copper zone on B.Cu, net /SW1OUT
- removed copper zone on F.Cu, net /SW1OUT
- removed copper zone on B.Cu, net /SW2OUT
- removed copper zone on F.Cu, net /SW2OUT
Other:
- board size 72 x 69 mm -> 152.4 x 76.2 mm

Commit message: layout starting to take shape
Parts:
- added H5: M4 4.3mm, MountingHole:MountingHole_4.3mm_M4, F.Cu at (151.2, 74.8)
- added H6: M4 4.3mm, MountingHole:MountingHole_4.3mm_M4, F.Cu at (151.2, 135.8)
- added U2: ACS71240LLCBTR-050B3, Package_SO:SOIC-8_3.9x4.9mm_P1.27mm, F.Cu at (197.0, 109.9)
- J1: footprint PCM_SparkFun-Connector:1x05_P2.54mm_Locking -> Connector_PinHeader_2.54mm:PinHeader_1x05_P2.54mm_Vertical
- J2: footprint PCM_SparkFun-Connector:1x04_P2.54mm_Locking -> Connector_PinHeader_2.54mm:PinHeader_1x04_P2.54mm_Vertical
- moved CIN1 118.2 mm to (184.5, 127.1)
- moved C5V2 118.2 mm to (192.2, 116.9)
- moved C5V3 118.2 mm to (192.2, 119.9)
- moved L1 118.2 mm to (185.6, 120.2)
- moved U3 118.2 mm to (190.0, 127.4)
- moved C15 112.8 mm to (173.6, 119.7)
- moved CIN2 112.8 mm to (173.6, 122.2)
- moved RFBT1 112.8 mm to (173.6, 124.7)
- moved RRFBB1 112.8 mm to (173.6, 127.2)
- moved COUT3 68.0 mm to (184.3, 103.2), turned to 90 degrees
- moved COUT4 57.7 mm to (173.8, 103.2), turned to 90 degrees
- moved RGND3 57.3 mm to (176.7, 112.0), turned to -90 degrees
- moved RPD3 52.4 mm to (176.8, 103.2), turned to -90 degrees
- moved COUT5 48.0 mm to (163.6, 103.2), turned to 90 degrees
- moved R13 44.5 mm to (158.6, 127.8)
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- renumbered COUT3 to C5V2, COUT4 to C5V3, COUT5 to COUT3, COUT6 to COUT4, COUT7 to COUT5
Connections:
- net /SW0DEN renamed /SWDEN5
- net /SW0IN renamed /SWIN5
- net /SW0IS renamed /SWIS5
- net /SW2DEN renamed /SWDEN4
- net /SW2IN renamed /SWIN4
- net /SW2IS renamed /SWIS4
- net /SW3DEN renamed /SWDEN3
- net /SW3IN renamed /SWIN3
- net /SW3IS renamed /SWIS3
- D1 pad 2: +12V -> /VBAT
- J3 pad 1: unconnected-(J3-Pin_1-Pad1) -> /SWOUT2
- J3 pad 3: unconnected-(J3-Pin_3-Pad3) -> /SWOUT1
- J3 pad 5: unconnected-(J3-Pin_5-Pad5) -> /SWOUT0
- J4 pad 1: +12V -> /VBAT
- J4 pad 2: +12V -> /VBAT
- J5 pad 1: unconnected-(J5-Pin_1-Pad1) -> /SWOUT3
- J5 pad 3: unconnected-(J5-Pin_3-Pad3) -> /SWOUT4
- J5 pad 5: unconnected-(J5-Pin_5-Pad5) -> /SWOUT5
- U1 pad 11: unconnected-(U1-PA4-Pad11) -> /IS_TOT
Routing:
- net +5V: track 47.7 -> 27.0 mm, vias 2 -> 1
- net +3.3V: track 69.6 -> 51.3 mm
- net GND: track 90.3 -> 106.9 mm, vias 23 -> 20
- net /VS: track 20.5 -> 6.55 mm
- net +12V: vias 120 -> 240
- added copper zone on B.Cu, net /VBAT
- added copper zone on F.Cu, net /VBAT
Other:
- board size 152.4 x 76.2 mm -> 107.7 x 76.2 mm
- board text added: "(C) 2026 G MCLELLAN SIX WAY HIGH SIDE SMART SWITCH EXT FUSING REQUIRED"
- board text added: "SW3+"
- board text added: "SW4+"
- board text added: "SW5+"
- board text removed: "(C) 2026 G MCLELLAN TRIPLE HIGH SIDE SMART SWITCH EXT FUSING REQUIRED"

Commit message: layout work continues
Parts:
- added CVS3: 68n, Capacitor_SMD:C_0603_1608Metric_Pad1.08x0.95mm_HandSolder, F.Cu at (184.3, 109.8)
- added CVS4: 68n, Capacitor_SMD:C_0603_1608Metric_Pad1.08x0.95mm_HandSolder, F.Cu at (173.8, 109.8)
- added CVS5: 68n, Capacitor_SMD:C_0603_1608Metric_Pad1.08x0.95mm_HandSolder, F.Cu at (163.6, 109.8)
- moved R15 31.8 mm to (182.8, 112.2), turned to 90 degrees
- moved R14 27.9 mm to (179.8, 112.2), turned to 90 degrees
- moved R17 27.7 mm to (169.3, 112.2), turned to 90 degrees
- moved R22 25.8 mm to (181.3, 112.2), turned to 90 degrees
- moved R13 25.1 mm to (178.3, 112.2), turned to -90 degrees
- moved R16 24.8 mm to (167.8, 112.2), turned to 90 degrees
- moved R24 23.1 mm to (162.1, 112.2), turned to 90 degrees
- moved R23 22.6 mm to (172.3, 112.2), turned to 90 degrees
- moved R21 15.7 mm to (160.6, 112.2), turned to 90 degrees
- moved R20 13.6 mm to (159.1, 112.2), turned to 90 degrees
- moved R19 11.8 mm to (157.6, 112.2), turned to 90 degrees
- moved R18 11.2 mm to (170.8, 112.2), turned to 90 degrees
- moved RGND3 0.25 mm to (176.8, 112.2)
- moved RGND5 0.25 mm to (156.1, 112.2)
- moved RGND4 0.23 mm to (166.3, 112.2)

Commit message: lots of work to do still
Parts:
- removed H4: M4 4.3mm, MountingHole:MountingHole_4.3mm_M4
- U1: value STM32G0B1KBTx -> STM32G0B1CCTx; footprint Package_QFP:LQFP-32_7x7mm_P0.8mm -> Package_QFP:LQFP-48_7x7mm_P0.5mm
- moved J1 13.3 mm to (186.6, 138.4), turned to 90 degrees
- moved CNRST1 8.72 mm to (212.9, 119.9), turned to 0 degrees
- moved CSTM1 3.03 mm to (211.9, 121.5)
- moved U1 2.18 mm to (206.2, 127.5), turned to 0 degrees
- moved CSTM2 1.96 mm to (210.8, 123.0)
Connections:
- J1 pad 1: +3.3V -> /NRST
- J1 pad 2: /NRST -> +3.3V
- J1 pad 3: /SWCLK -> /SWDIO
- J1 pad 4: /SWDIO -> /SWCLK
- U1 pad 10: /VS -> /NRST
- U1 pad 11: /IS_TOT -> /SWIS1
- U1 pad 12: unconnected-(U1-PA5-Pad12) -> /SWIS0
- U1 pad 13: unconnected-(U1-PA6-Pad13) -> /SWDEN0
- U1 pad 14: unconnected-(U1-PA7-Pad14) -> /SWIN0
- U1 pad 19: /USART1_TX -> /CAN_RX
- U1 pad 20: unconnected-(U1-PC6-Pad20) -> /CAN_TX
- U1 pad 21: /USART1_RX -> unconnected-(U1-PB2-Pad21)
- U1 pad 22: /CAN1_RX -> unconnected-(U1-PB10-Pad22)
- U1 pad 23: /CAN1_TX -> unconnected-(U1-PB11-Pad23)
- U1 pad 24: /SWDIO -> unconnected-(U1-PB12-Pad24)
- U1 pad 25: /SWCLK -> /USART1_TX
- U1 pad 26: unconnected-(U1-PA15-Pad26) -> /USART1_RX
- U1 pad 27: /SWDEN2 -> unconnected-(U1-PB15-Pad27)
- U1 pad 28: /SWIN2 -> unconnected-(U1-PA8-Pad28)
- U1 pad 29: /SWDEN1 -> unconnected-(U1-PA9/UCPD1_DBCC1-Pad29)
- U1 pad 30: /SWIN1 -> unconnected-(U1-PC6-Pad30)
- U1 pad 31: /SWDEN0 -> unconnected-(U1-PC7-Pad31)
- U1 pad 32: /SWIN0 -> unconnected-(U1-PA10/UCPD1_DBCC2-Pad32)
- U1 pad 4: +3.3V -> unconnected-(U1-VBAT-Pad4)
- U1 pad 5: GND -> +3.3V
- U1 pad 6: /NRST -> +3.3V
- U1 pad 7: /SWIS1 -> GND
- U1 pad 8: /SWIS2 -> unconnected-(U1-PF0-Pad8)
- U1 pad 9: /SWIS0 -> unconnected-(U1-PF1-Pad9)
- U4 pad 1: /CAN1_TX -> /CAN_TX
- U4 pad 4: /CAN1_RX -> /CAN_RX
Routing:
- net +3.3V: track 51.3 -> 21.2 mm, vias 1 -> 0
- net /SWIS2: track 40.2 -> 16.8 mm, vias 2 -> 1
- net /SWIS0: track 23.9 -> 1.53 mm, vias 2 -> 0
- net +5V: track 27.0 -> 7.61 mm
- net /SWIS1: track 31.4 -> 14.3 mm, vias 2 -> 1
- net /SWDIO: track 16.8 -> 0.00 mm
- net /NRST: track 16.7 -> 0.00 mm, vias 2 -> 0
- net /SWCLK: track 15.9 -> 0.00 mm, vias 2 -> 0
- net /SWIN2: track 33.3 -> 19.5 mm
- net /SWDEN0: track 15.6 -> 2.76 mm
- net /SWIN0: track 14.6 -> 2.55 mm
- net /CAN_RX: track 0.00 -> 10.0 mm
- net /CAN1_RX: track 10.0 -> 0.00 mm
- net /SWDEN2: track 35.2 -> 26.5 mm
- net /CAN_TX: track 0.00 -> 8.24 mm
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
Commit message: making progress on layout and routing
Parts:
- added CACS1: 100n, Capacitor_SMD:C_0603_1608Metric_Pad1.08x0.95mm_HandSolder, F.Cu at (200.8, 112.3)
- added CIST1: 100n, Capacitor_SMD:C_0603_1608Metric_Pad1.08x0.95mm_HandSolder, F.Cu at (198.7, 116.7)
- added RFAULT1: 10K, Resistor_SMD:R_0603_1608Metric_Pad0.98x0.95mm_HandSolder, F.Cu at (197.7, 115.1)
- U2: value ACS71240LLCBTR-050B3 -> ACS712
- moved CIN2 25.4 mm to (197.0, 131.9)
- moved CB1 20.8 mm to (191.0, 131.0)
- moved CNRST1 15.1 mm to (201.1, 129.4), turned to 180 degrees
- moved CIN1 14.1 mm to (196.6, 134.3)
- moved RFB1 13.7 mm to (187.0, 127.5), turned to -90 degrees
- moved RFB2 11.9 mm to (185.5, 127.5), turned to -90 degrees
- moved CSTM1 11.6 mm to (200.9, 125.0), turned to 180 degrees
- moved CSTM2 10.4 mm to (201.1, 126.8), turned to 180 degrees
- moved C5V2 9.94 mm to (184.8, 123.6), turned to -90 degrees
- moved L1 8.16 mm to (191.7, 125.6)
- moved C5V3 6.49 mm to (186.8, 123.6), turned to -90 degrees
- moved U3 6.33 mm to (191.2, 133.6)
- moved U1 2.24 mm to (208.4, 127.6)
- moved U2 0.54 mm to (197.0, 110.4)
- moved J5 0.40 mm to (180.2, 87.5)
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- renumbered C15 to CB1, RFBT1 to RFB1, RRFBB1 to RFB2
Connections:
- net Net-(U3-FB) renamed /FB
- U1 pad 11: /SWIS1 -> unconnected-(U1-PA0-Pad11)
- U1 pad 12: /SWIS0 -> unconnected-(U1-PA1-Pad12)
- U1 pad 13: /SWDEN0 -> unconnected-(U1-PA2-Pad13)
- U1 pad 14: /SWIN0 -> unconnected-(U1-PA3-Pad14)
- U2 pad 6: unconnected-(U2-FILTER-Pad6) -> /IFAULT
Routing:
- net GND: track 101.8 -> 172.7 mm, vias 16 -> 45
- net /SWDEN2: track 26.5 -> 0.00 mm
- net /SWIN2: track 19.5 -> 0.00 mm
- net /SWDEN1: track 18.0 -> 0.00 mm
- net /SWIN1: track 16.8 -> 0.00 mm
- net /SWIS2: track 16.8 -> 0.00 mm, vias 1 -> 0
- net /SWIS1: track 14.3 -> 0.00 mm, vias 1 -> 0
- net /FB: track 0.00 -> 10.2 mm
- net +5V: track 7.61 -> 15.2 mm
- net /CAN_RX: track 10.0 -> 16.1 mm
- net +3.3V: track 21.2 -> 26.8 mm, vias 0 -> 1
- net /IS_TOT: track 0.00 -> 3.93 mm
- net /SWIS_PD5: track 0.00 -> 3.90 mm
- net /SWIS_PD3: track 0.00 -> 3.90 mm
- net /SWIS_PD4: track 0.00 -> 3.88 mm
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- added copper zone on F.Cu, net /SW
- added copper zone on B.Cu, net /SWOUT3
- added copper zone on F.Cu, net /SWOUT3
- added copper zone on B.Cu, net /SWOUT4
- added copper zone on F.Cu, net /SWOUT4
- added copper zone on B.Cu, net /SWOUT5
- added copper zone on F.Cu, net /SWOUT5
- added copper zone on F.Cu, net GND
Other:
- board text added: "3V3 TX RX GND"
- board text added: "RST 3V3 DIO CLK GND"

Commit message: great progress with routing so far
Parts:
- U1: value STM32G0B1CCTx -> STM32G0B1RCTx; footprint Package_QFP:LQFP-48_7x7mm_P0.5mm -> Package_QFP:LQFP-64_10x10mm_P0.5mm
- moved CNRST1 19.5 mm to (219.6, 123.2), turned to 0 degrees
- moved CSTM1 19.2 mm to (219.8, 127.6), turned to 0 degrees
- moved CSTM2 18.5 mm to (219.6, 125.8), turned to 0 degrees
- moved CDIV1 10.5 mm to (206.7, 112.2)
- moved RVDIV1 10.5 mm to (203.7, 112.2)
- moved RVDIV2 10.5 mm to (205.2, 112.2)
- moved U1 2.78 mm to (209.8, 125.2), turned to 180 degrees
Connections:
- U1 pad 10: /NRST -> unconnected-(U1-PF0-Pad10)
- U1 pad 12: unconnected-(U1-PA1-Pad12) -> /NRST
- U1 pad 17: unconnected-(U1-PA6-Pad17) -> /SWIS2
- U1 pad 18: unconnected-(U1-PA7-Pad18) -> /SWDEN2
- U1 pad 19: /CAN_RX -> /SWIN2
- U1 pad 20: /CAN_TX -> /SWIS1
- U1 pad 21: unconnected-(U1-PB2-Pad21) -> /SWDEN1
- U1 pad 22: unconnected-(U1-PB10-Pad22) -> /SWIN1
- U1 pad 23: unconnected-(U1-PB11-Pad23) -> /SWIS0
- U1 pad 24: unconnected-(U1-PB12-Pad24) -> /SWDEN0
- U1 pad 25: /USART1_TX -> /SWIN0
- U1 pad 26: /USART1_RX -> /VS
- U1 pad 27: unconnected-(U1-PB15-Pad27) -> /IS_TOT
- U1 pad 5: +3.3V -> unconnected-(U1-PC15-Pad5)
- U1 pad 6: +3.3V -> unconnected-(U1-VBAT-Pad6)
- U1 pad 7: GND -> +3.3V
- U1 pad 8: unconnected-(U1-PF0-Pad8) -> +3.3V
- U1 pad 9: unconnected-(U1-PF1-Pad9) -> GND
Routing:
- net /SWIS2: track 0.00 -> 25.8 mm
- net /SWDEN2: track 0.00 -> 25.3 mm
- net /SWIN2: track 0.00 -> 24.2 mm
- net /SWIS1: track 0.00 -> 18.0 mm
- net /SWDEN1: track 0.00 -> 15.5 mm
- net /SWIN1: track 0.00 -> 14.5 mm
- net /IS_TOT: track 3.93 -> 16.9 mm
- net /VS: track 0.00 -> 10.5 mm
- net /SWIS0: track 0.00 -> 9.30 mm
- net /SWDEN0: track 0.00 -> 7.27 mm
- net /SWIN0: track 0.00 -> 6.85 mm
- net /CAN_RX: track 16.1 -> 10.3 mm
- net /CAN_TX: track 8.31 -> 3.37 mm
- net GND: track 172.7 -> 170.0 mm, vias 45 -> 46
- net /USART1_RX: track 1.50 -> 0.00 mm, vias 1 -> 0
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
Commit message: signals routed, next is power
Parts:
- J2: value USART1 -> USART2
- moved R9 1.51 mm to (225.3, 112.2)
- moved R11 1.50 mm to (213.5, 112.2)
- moved R12 1.50 mm to (215.0, 112.2)
- moved R15 1.50 mm to (181.3, 112.2)
- moved R22 1.50 mm to (182.8, 112.2)
- moved R5 1.50 mm to (223.8, 112.2)
- moved CSTM1 0.68 mm to (219.2, 127.3)
- moved CSTM2 0.65 mm to (219.0, 125.5)
- moved CNRST1 0.63 mm to (219.0, 123.4)
- moved CIST1 0.30 mm to (198.7, 117.0)
- moved RPD0 0.23 mm to (208.9, 103.4)
- moved COUT2 0.10 mm to (238.1, 103.5)
- moved CVS1 0.06 mm to (226.8, 110.1)
Connections:
- J2 pad 2: /USART1_TX -> /USART2_TX
- J2 pad 3: /USART1_RX -> /USART2_RX
- U1 pad 28: unconnected-(U1-PB1-Pad28) -> /SWIS3
- U1 pad 29: unconnected-(U1-PB2-Pad29) -> /SWIS4
- U1 pad 30: unconnected-(U1-PB10-Pad30) -> /SWIS5
- U1 pad 33: unconnected-(U1-PB13-Pad33) -> /SWDEN3
- U1 pad 34: unconnected-(U1-PB14-Pad34) -> /SWIN3
- U1 pad 35: unconnected-(U1-PB15-Pad35) -> /SWDEN4
- U1 pad 36: unconnected-(U1-PA8-Pad36) -> /SWIN4
- U1 pad 38: unconnected-(U1-PC6-Pad38) -> /SWDEN5
- U1 pad 39: unconnected-(U1-PC7-Pad39) -> /SWIN5
- U1 pad 45: unconnected-(U1-PA13-Pad45) -> /SWDIO
- U1 pad 46: unconnected-(U1-PA14-Pad46) -> /SWCLK
- U1 pad 50: unconnected-(U1-PD0-Pad50) -> /CAN_RX
- U1 pad 51: unconnected-(U1-PD1-Pad51) -> /CAN_TX
- U1 pad 55: unconnected-(U1-PD5-Pad55) -> /USART2_TX
- U1 pad 56: unconnected-(U1-PD6-Pad56) -> /USART2_RX
Routing:
- net /SWIN5: track 0.00 -> 53.6 mm, vias 0 -> 2
- net /NRST: track 0.00 -> 51.6 mm
- net /SWIS5: track 0.00 -> 51.2 mm, vias 0 -> 2
- net /SWDEN5: track 0.00 -> 51.2 mm, vias 0 -> 2
- net /SWIN4: track 0.00 -> 42.7 mm, vias 0 -> 2
- net /SWIS4: track 0.00 -> 41.3 mm, vias 0 -> 2
- net /SWDEN4: track 0.00 -> 41.0 mm, vias 0 -> 2
- net +3.3V: track 26.8 -> 64.0 mm, vias 1 -> 3
- net /SWIN3: track 0.00 -> 32.2 mm, vias 0 -> 2
- net /SWIS3: track 0.00 -> 31.1 mm, vias 0 -> 2
- net /SWDEN3: track 0.00 -> 30.2 mm, vias 0 -> 2
- net /SWDIO: track 0.00 -> 27.6 mm
- net /SWCLK: track 0.00 -> 23.6 mm
- net /CAN_RX: track 10.3 -> 20.5 mm
- net /USART2_TX: track 0.00 -> 9.39 mm
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
Commit message: everything is routed, drc passed
Parts:
- added D2: STAT1, LED_SMD:LED_0805_2012Metric_Pad1.15x1.40mm_HandSolder, F.Cu at (100.4, 82.6)
- added D3: STAT2, LED_SMD:LED_0805_2012Metric_Pad1.15x1.40mm_HandSolder, F.Cu at (103.0, 82.6)
- added R25: 1K0, Resistor_SMD:R_0603_1608Metric_Pad0.98x0.95mm_HandSolder, F.Cu at (100.5, 86.4)
- added R26: 1K0, Resistor_SMD:R_0603_1608Metric_Pad0.98x0.95mm_HandSolder, F.Cu at (103.0, 86.4)
- moved CIN2 120.3 mm to (88.5, 80.0), turned to 90 degrees
- moved CIN1 118.6 mm to (91.0, 80.4), turned to 90 degrees
- moved L1 117.7 mm to (81.2, 84.8), turned to 90 degrees
- moved CB1 113.8 mm to (86.7, 85.5), turned to 90 degrees
- moved U3 112.8 mm to (89.2, 85.3), turned to 90 degrees
- moved C5V3 112.8 mm to (79.2, 89.7), turned to 0 degrees
- moved RFB1 110.6 mm to (83.1, 89.5), turned to 0 degrees
- moved C5V2 110.3 mm to (79.2, 91.7), turned to 0 degrees
- moved RFB2 108.7 mm to (83.1, 91.0), turned to 0 degrees
- moved C3V1 103.3 mm to (127.0, 93.4)
- moved CACS1 103.3 mm to (108.0, 66.9)
- moved CIST1 103.3 mm to (106.0, 71.6)
- moved COUT3 103.3 mm to (91.5, 57.8)
- moved COUT4 103.3 mm to (81.0, 57.8)
- moved CVS3 103.3 mm to (91.5, 64.4)
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Connections:
- U1 pad 40: unconnected-(U1-PD8-Pad40) -> /STAT1
- U1 pad 41: unconnected-(U1-PD9-Pad41) -> /STAT2
Routing:
- net +5V: track 15.2 -> 117.2 mm, vias 1 -> 3
- net +3.3V: track 64.0 -> 110.2 mm, vias 3 -> 4
- net /STAT1: track 0.00 -> 12.7 mm
- net /STAT2: track 0.00 -> 9.54 mm
- net GND: track 170.2 -> 172.4 mm, vias 53 -> 65
- net Net-(D3-K): track 0.00 -> 1.83 mm
- net Net-(D2-K): track 0.00 -> 1.78 mm
